Commit message: properly merged effort controller

File: src/turtlebot3/turtlebot3_description/urdf/turtlebot3_waffle_pi_effort_controller.gazebo.xacro (robot description, xacro)
@@ -8,6 +8,6 @@
   </gazebo>
   <gazebo reference="wheel_left_link">
-    <mu1>0.1</mu1>
-    <mu2>0.1</mu2>
+    <mu1>10</mu1>
+    <mu2>10</mu2>
     <kp>500000.0</kp>
     <kd>10.0</kd>
@@ -18,6 +18,6 @@
   </gazebo>
   <gazebo reference="wheel_right_link">
-    <mu1>0.1</mu1>
-    <mu2>0.1</mu2>
+    <mu1>10</mu1>
+    <mu2>10</mu2>
     <kp>500000.0</kp>
     <kd>10.0</kd>
@@ -52,9 +52,9 @@
     <material>Gazebo/Grey</material>
   </gazebo>
-  <!-- <gazebo>
+  <gazebo>
     <plugin name="gazebo_ros_control" filename="libgazebo_ros_control.so">
       <robotSimType>gazebo_ros_control/DefaultRobotHWSim</robotSimType>
     </plugin>
-  </gazebo> -->
+  </gazebo>
   <!-- <gazebo>
     <plugin name="gazebo_ros_control" filename="libgazebo_ros_control.so">

File: src/turtlebot3/turtlebot3_description/urdf/turtlebot3_waffle_pi_effort_controller.urdf.xacro (robot description, xacro)
@@ -36,5 +36,5 @@
     <origin xyz="0.0 0.144 0.023" rpy="-1.57 0 0"/>
     <axis xyz="0 0 1"/>
-    <limit effort="1" velocity="0" lower="-2.61799387799" upper="1.98394848567"/>
+    <limit effort="1.0" velocity="0.5"/>
   </joint>
   <link name="wheel_left_link">
@@ -65,5 +65,5 @@
     <origin xyz="0.0 -0.144 0.023" rpy="-1.57 0 0"/>
     <axis xyz="0 0 1"/>
-    <limit effort="1" velocity="0" lower="-2.61799387799" upper="1.98394848567"/>
+    <limit effort="1.0" velocity="0.5"/>
   </joint>
   <link name="wheel_right_link">

Commit message: the effort controller is actually working

File: src/turtlebot3/turtlebot3_description/urdf/turtlebot3_waffle_pi_effort_controller.gazebo.xacro (robot description, xacro)
@@ -8,6 +8,6 @@
   </gazebo>
   <gazebo reference="wheel_left_link">
-    <mu1>10</mu1>
-    <mu2>10</mu2>
+    <mu1>0.5</mu1>
+    <mu2>0.5</mu2>
     <kp>500000.0</kp>
     <kd>10.0</kd>
@@ -18,6 +18,6 @@
   </gazebo>
   <gazebo reference="wheel_right_link">
-    <mu1>10</mu1>
-    <mu2>10</mu2>
+    <mu1>0.5</mu1>
+    <mu2>0.5</mu2>
     <kp>500000.0</kp>
     <kd>10.0</kd>
@@ -29,5 +29,5 @@
   <gazebo reference="caster_back_right_link">
     <mu1>0.1</mu1>
-    <mu2>0.1</mu2>
+    <mu2>0.1  </mu2>
     <kp>1000000.0</kp>
     <kd>100.0</kd>

File: src/turtlebot3/turtlebot3_description/urdf/turtlebot3_waffle_pi_effort_controller.urdf.xacro (robot description, xacro)
@@ -36,5 +36,5 @@
     <origin xyz="0.0 0.144 0.023" rpy="-1.57 0 0"/>
     <axis xyz="0 0 1"/>
-    <limit effort="1.0" velocity="0.5"/>
+    <limit effort="3.0" velocity="2.57"/>
   </joint>
   <link name="wheel_left_link">
@@ -65,5 +65,5 @@
     <origin xyz="0.0 -0.144 0.023" rpy="-1.57 0 0"/>
     <axis xyz="0 0 1"/>
-    <limit effort="1.0" velocity="0.5"/>
+    <limit effort="3.0" velocity="2.57"/>
   </joint>
   <link name="wheel_right_link">

Commit message: sim works, odom pub works

File: src/turtlebot3/turtlebot3_description/urdf/turtlebot3_waffle_pi_effort_controller.gazebo.xacro (robot description, xacro)
@@ -8,6 +8,6 @@
   </gazebo>
   <gazebo reference="wheel_left_link">
-    <mu1>0.5</mu1>
-    <mu2>0.5</mu2>
+    <mu1>0.9</mu1>
+    <mu2>0.9</mu2>
     <kp>500000.0</kp>
     <kd>10.0</kd>
@@ -18,6 +18,6 @@
   </gazebo>
   <gazebo reference="wheel_right_link">
-    <mu1>0.5</mu1>
-    <mu2>0.5</mu2>
+    <mu1>0.9</mu1>
+    <mu2>0.9</mu2>
     <kp>500000.0</kp>
     <kd>10.0</kd>
@@ -87,5 +87,5 @@
       <serviceName>imu_service</serviceName>
       <gaussianNoise>0.0</gaussianNoise>
-      <updateRate>200</updateRate>
+      <updateRate>100</updateRate>
       <imu>
         <noise>

File: src/turtlebot3/turtlebot3_description/urdf/turtlebot3_waffle_pi_effort_controller.urdf.xacro (robot description, xacro)
@@ -36,5 +36,5 @@
     <origin xyz="0.0 0.144 0.023" rpy="-1.57 0 0"/>
     <axis xyz="0 0 1"/>
-    <limit effort="3.0" velocity="2.57"/>
+    <limit effort="10.0" velocity="8.6"/>
   </joint>
   <link name="wheel_left_link">
@@ -65,5 +65,5 @@
     <origin xyz="0.0 -0.144 0.023" rpy="-1.57 0 0"/>
     <axis xyz="0 0 1"/>
-    <limit effort="3.0" velocity="2.57"/>
+    <limit effort="10.0" velocity="8.6"/>
   </joint>
   <link name="wheel_right_link">
